File: Schematics/Main_Board.sch (EAGLE design)
At the start: 84 parts, among them IC1 LM317MBSTT3, IC2 LM317MBSTT3, Q1 32.768kHz, X1 MINI-USB-SHIELD-UX60-MB-5ST, X2 RJ45

Commit message: Mostly updates with some sensor stuff
Connections:
- new net N$42: U$1.4, X2.1
- net +5V: now also X2.5; no longer X2.1
- net GND: now also X2.6; no longer X2.5
- net N$20: now also X2.7; no longer X2.6
- net N$21: now also X2.8; no longer X2.7
- net N$22: no longer X2.8
Other:
- note added: "+ Analog Input"
- note added: "- Analog Input"
- note added: "2"
- note added: "4/28/2014"
- note removed: "Analog Input"
- note removed: "Unspecified use is tied to unused GPIO"
- moved on the sheet: C14
Changed lines of the file:
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@@
 <part name="P+1" library="supply1" deviceset="+5V" device=""/>
 <part name="+3V1" library="supply1" deviceset="+3V3" device=""/>
-<part name="P+2" library="supply1" deviceset="+5V" device=""/>
 <part name="GND21" library="supply1" deviceset="GND" device=""/>
 <part name="R4" library="rcl" deviceset="R-US_" device="R0603" value="22"/>
@@
 <part name="GND33" library="supply1" deviceset="GND" device=""/>
 <part name="SUPPLY8" library="supply2" deviceset="V+" device=""/>
+<part name="P+2" library="supply1" deviceset="+5V" device=""/>
+<part name="FRAME1" library="frames" deviceset="FRAME_B_L" device=""/>
 </parts>
 <sheets>
@@
 <wire x1="101.6" y1="116.84" x2="101.6" y2="81.28" width="0.1524" layer="97"/>
 <wire x1="101.6" y1="81.28" x2="22.86" y2="81.28" width="0.1524" layer="97"/>
-<wire x1="22.86" y1="81.28" x2="22.86" y2="116.84" width="0.1524" layer="97"/>
 <text x="50.8" y="111.76" size="1.778" layer="97">INTERFACE TO SENSOR</text>
 <wire x1="129.54" y1="43.18" x2="129.54" y2="-30.48" width="0.1524" layer="97"/>
@@
 <text x="38.1" y="88.9" size="1.778" layer="97">+Comparator input</text>
 <text x="38.1" y="86.36" size="1.778" layer="97">-Comparator input</text>
-<text x="35.56" y="91.44" size="1.778" layer="97">Analog Input</text>
-<text x="73.66" y="91.44" size="1.778" layer="97">I2C:SCL</text>
-<text x="71.12" y="86.36" size="1.778" layer="97">I2C:SDA</text>
-<text x="78.74" y="96.52" size="1.778" layer="97">Unspecified use is tied to unused GPIO</text>
+<text x="35.56" y="91.44" size="1.778" layer="97">- Analog Input</text>
+<text x="78.74" y="96.52" size="1.778" layer="97">I2C:SCL</text>
+<text x="76.2" y="91.44" size="1.778" layer="97">I2C:SDA</text>
 <text x="-142.24" y="45.72" size="1.778" layer="97" rot="R90">L1</text>
 <text x="-132.08" y="43.18" size="1.778" layer="97" rot="R90">4.7uH</text>
@@
 <text x="-111.76" y="63.5" size="1.778" layer="97">LTC3534</text>
 <text x="-111.76" y="2.54" size="1.778" layer="97">LTC3534</text>
-<text x="27.94" y="96.52" size="1.778" layer="97">Analog Power</text>
+<wire x1="22.86" y1="81.28" x2="22.86" y2="116.84" width="0.1524" layer="97"/>
+<text x="50.8" y="83.82" size="1.778" layer="97">Analog Power</text>
+<text x="33.02" y="96.52" size="1.778" layer="97">+ Analog Input</text>
+<text x="213.36" y="-83.82" size="2.54" layer="94">2</text>
+<text x="134.62" y="-91.44" size="2.54" layer="94">4/28/2014</text>
 </plain>
 <instances>
@@
 <instance part="P+1" gate="1" x="10.16" y="66.04"/>
 <instance part="+3V1" gate="G$1" x="12.7" y="15.24"/>
-<instance part="P+2" gate="1" x="48.26" y="101.6"/>
-<instance part="GND21" gate="1" x="66.04" y="81.28"/>
+<instance part="GND21" gate="1" x="78.74" y="81.28"/>
 <instance part="R4" gate="G$1" x="134.62" y="15.24" smashed="yes" rot="R90">
 <attribute name="NAME" x="133.1214" y="11.43" size="1.778" layer="95" rot="R90"/>
@@
 </instance>
 <instance part="GND22" gate="1" x="121.92" y="20.32"/>
-<instance part="C14" gate="G$1" x="33.02" y="91.44" rot="R180"/>
+<instance part="C14" gate="G$1" x="73.66" y="83.82" rot="R270"/>
 <instance part="R12" gate="G$1" x="96.52" y="106.68" smashed="yes" rot="R90">
 <attribute name="NAME" x="100.1014" y="107.95" size="1.778" layer="95" rot="R90"/>
@@
 <instance part="C15" gate="G$1" x="45.72" y="53.34" rot="R180"/>
 <instance part="GND23" gate="1" x="45.72" y="48.26"/>
-<instance part="P+6" gate="1" x="45.72" y="66.04"/>
+<instance part="P+6" gate="1" x="45.72" y="63.5"/>
 <instance part="P+7" gate="1" x="45.72" y="38.1"/>
 <instance part="C16" gate="G$1" x="45.72" y="27.94" rot="R180"/>
@@
 <instance part="GND33" gate="1" x="-99.06" y="93.98"/>
 <instance part="SUPPLY8" gate="1" x="-99.06" y="121.92"/>
+<instance part="P+2" gate="1" x="27.94" y="91.44"/>
+<instance part="FRAME1" gate="G$1" x="-205.74" y="-93.98"/>
+<instance part="FRAME1" gate="G$2" x="119.38" y="-91.44" smashed="yes">
+<attribute name="SHEET" x="205.74" y="-90.17" size="2.54" layer="94" font="vector"/>
+<attribute name="DRAWING_NAME" x="137.16" y="-72.39" size="2.54" layer="94" font="vector"/>
+</instance>
 </instances>
 <busses>
@@
 <pinref part="R11" gate="G$1" pin="1"/>
 <wire x1="121.92" y1="22.86" x2="121.92" y2="25.4" width="0.1524" layer="91"/>
-</segment>
-<segment>
-<pinref part="GND21" gate="1" pin="GND"/>
-<pinref part="X2" gate="G$1" pin="5"/>
-<wire x1="66.04" y1="83.82" x2="66.04" y2="96.52" width="0.1524" layer="91"/>
-<pinref part="C14" gate="G$1" pin="1"/>
-<wire x1="33.02" y1="88.9" x2="33.02" y2="83.82" width="0.1524" layer="91"/>
-<wire x1="33.02" y1="83.82" x2="66.04" y2="83.82" width="0.1524" layer="91"/>
-<junction x="66.04" y="83.82"/>
 </segment>
 <segment>
@@
 <pinref part="GND33" gate="1" pin="GND"/>
 </segment>
+<segment>
+<pinref part="GND21" gate="1" pin="GND"/>
+<pinref part="C14" gate="G$1" pin="1"/>
+<wire x1="78.74" y1="83.82" x2="76.2" y2="83.82" width="0.1524" layer="91"/>
+<wire x1="76.2" y1="83.82" x2="76.2" y2="88.9" width="0.1524" layer="91"/>
+<junction x="76.2" y="83.82"/>
+<wire x1="76.2" y1="88.9" x2="68.58" y2="88.9" width="0.1524" layer="91"/>
+<pinref part="X2" gate="G$1" pin="6"/>
+<wire x1="68.58" y1="88.9" x2="68.58" y2="96.52" width="0.1524" layer="91"/>
+</segment>
 </net>
 <net name="N$11" class="0">
@@
 </segment>
 <segment>
-<wire x1="55.88" y1="96.52" x2="48.26" y2="96.52" width="0.1524" layer="91"/>
-<pinref part="P+2" gate="1" pin="+5V"/>
-<pinref part="X2" gate="G$1" pin="1"/>
-<wire x1="48.26" y1="96.52" x2="48.26" y2="99.06" width="0.1524" layer="91"/>
-<pinref part="C14" gate="G$1" pin="2"/>
-<wire x1="33.02" y1="96.52" x2="48.26" y2="96.52" width="0.1524" layer="91"/>
-<junction x="48.26" y="96.52"/>
-</segment>
-<segment>
 <pinref part="R14" gate="G$1" pin="2"/>
 <pinref part="P+3" gate="1" pin="+5V"/>
@@
 <wire x1="53.34" y1="58.42" x2="45.72" y2="58.42" width="0.1524" layer="91"/>
 <pinref part="P+6" gate="1" pin="+5V"/>
-<wire x1="45.72" y1="63.5" x2="45.72" y2="58.42" width="0.1524" layer="91"/>
+<wire x1="45.72" y1="60.96" x2="45.72" y2="58.42" width="0.1524" layer="91"/>
 <junction x="45.72" y="58.42"/>
 </segment>
@@
 <wire x1="45.72" y1="33.02" x2="45.72" y2="35.56" width="0.1524" layer="91"/>
 <junction x="45.72" y="33.02"/>
+</segment>
+<segment>
+<pinref part="C14" gate="G$1" pin="2"/>
+<pinref part="X2" gate="G$1" pin="5"/>
+<wire x1="68.58" y1="83.82" x2="66.04" y2="83.82" width="0.1524" layer="91"/>
+<wire x1="66.04" y1="83.82" x2="66.04" y2="96.52" width="0.1524" layer="91"/>
+<wire x1="66.04" y1="83.82" x2="27.94" y2="83.82" width="0.1524" layer="91"/>
+<junction x="66.04" y="83.82"/>
+<wire x1="27.94" y1="83.82" x2="27.94" y2="88.9" width="0.1524" layer="91"/>
+<pinref part="P+2" gate="1" pin="+5V"/>
 </segment>
 </net>
@@
 <pinref part="U$1" gate="G$1" pin="43"/>
 <wire x1="88.9" y1="60.96" x2="91.44" y2="60.96" width="0.1524" layer="91"/>
-<wire x1="91.44" y1="60.96" x2="91.44" y2="86.36" width="0.1524" layer="91"/>
-<pinref part="X2" gate="G$1" pin="6"/>
-<wire x1="91.44" y1="86.36" x2="68.58" y2="86.36" width="0.1524" layer="91"/>
-<wire x1="68.58" y1="86.36" x2="68.58" y2="96.52" width="0.1524" layer="91"/>
+<wire x1="91.44" y1="60.96" x2="91.44" y2="91.44" width="0.1524" layer="91"/>
 <pinref part="R13" gate="G$1" pin="1"/>
-<wire x1="91.44" y1="101.6" x2="91.44" y2="86.36" width="0.1524" layer="91"/>
-<junction x="91.44" y="86.36"/>
+<pinref part="X2" gate="G$1" pin="7"/>
+<wire x1="91.44" y1="91.44" x2="91.44" y2="101.6" width="0.1524" layer="91"/>
+<wire x1="71.12" y1="96.52" x2="71.12" y2="91.44" width="0.1524" layer="91"/>
+<wire x1="71.12" y1="91.44" x2="91.44" y2="91.44" width="0.1524" layer="91"/>
+<junction x="91.44" y="91.44"/>
 </segment>
 </net>
@@
 <pinref part="U$1" gate="G$1" pin="42"/>
 <wire x1="88.9" y1="58.42" x2="96.52" y2="58.42" width="0.1524" layer="91"/>
-<wire x1="96.52" y1="58.42" x2="96.52" y2="91.44" width="0.1524" layer="91"/>
-<pinref part="X2" gate="G$1" pin="7"/>
-<wire x1="96.52" y1="91.44" x2="71.12" y2="91.44" width="0.1524" layer="91"/>
-<wire x1="71.12" y1="91.44" x2="71.12" y2="96.52" width="0.1524" layer="91"/>
+<wire x1="96.52" y1="58.42" x2="96.52" y2="96.52" width="0.1524" layer="91"/>
 <pinref part="R12" gate="G$1" pin="1"/>
-<wire x1="96.52" y1="101.6" x2="96.52" y2="91.44" width="0.1524" layer="91"/>
-<junction x="96.52" y="91.44"/>
+<pinref part="X2" gate="G$1" pin="8"/>
+<wire x1="96.52" y1="96.52" x2="96.52" y2="101.6" width="0.1524" layer="91"/>
+<wire x1="96.52" y1="96.52" x2="73.66" y2="96.52" width="0.1524" layer="91"/>
+<junction x="96.52" y="96.52"/>
 </segment>
 </net>
 <net name="N$22" class="0">
 <segment>
-<pinref part="X2" gate="G$1" pin="8"/>
-<wire x1="73.66" y1="96.52" x2="116.84" y2="96.52" width="0.1524" layer="91"/>
 <wire x1="116.84" y1="96.52" x2="116.84" y2="60.96" width="0.1524" layer="91"/>
 <wire x1="116.84" y1="60.96" x2="99.06" y2="60.96" width="0.1524" layer="91"/>
@@
 </segment>
 </net>
+<net name="N$42" class="0">
+<segment>
+<pinref part="U$1" gate="G$1" pin="4"/>
+<wire x1="53.34" y1="66.04" x2="35.56" y2="66.04" width="0.1524" layer="91"/>
+<wire x1="35.56" y1="66.04" x2="35.56" y2="96.52" width="0.1524" layer="91"/>
+<pinref part="X2" gate="G$1" pin="1"/>
+<wire x1="35.56" y1="96.52" x2="55.88" y2="96.52" width="0.1524" layer="91"/>
+</segment>
+</net>
