File: Schematics/LDO/Main_Board.sch (EAGLE design)
At the start: 88 parts, among them IC1 LM317MBSTT3, IC2 LM317MBSTT3, Q1 32.768kHz, X1 MINI-USB-SHIELD-UX60-MB-5ST, X2 RJ45

Commit message: Updates for pin assignments
Parts:
- removed C21, C22: 10pF, rcl:C-USC0805
- removed C23, C26: 330pF, rcl:C-USC0805
- removed C24, C25: 10uF, rcl:C-USC0805
- removed C27, C29: 33pf, rcl:C-USC0805
- removed C28, C30: 22uF, rcl:C-USC0805
- removed D5, D6, D7, D8: 1N5818-T, diode:1N5818-T
- removed L1, L2: 4.7uH, Inductor:SHEILDED_COIL
- removed LED1: GREEN, led:LED5MM
- removed LED3: GM1WA55311A, led:GM1WA55311A
- removed POWER_IN1: 6v, pinhead:PINHD-1X2
- removed R19: 200k, resistor:R-US_R1206
- removed R20, R23, R26: 10k, rcl:R-US_R0805
- removed R21: 15k, rcl:R-US_R0805
- removed R22, R24: 162k, rcl:R-US_R0805
- removed R25: 649k, rcl:R-US_R0805
- removed R27: 373k, rcl:R-US_R0805
- removed R28: 330, rcl:R-US_R0603
- removed U$3: SWITCHER, linear-technology-2:SWITCHER
- R16: value 200k -> 180; device resistor:R-US_R1206 -> rcl:R-US_R0603
- R17: value 10k -> 100; device rcl:R-US_R0805 -> rcl:R-US_R0603
- R18: value 15k -> 100; device rcl:R-US_R0805 -> rcl:R-US_R0603
- U$2: value SWITCHER -> RGB_LED; device linear-technology-2:SWITCHER -> RGB_LED:RGB_LED
Connections:
- removed net N$27: R17.1, U$2.PWM
- removed net N$28: D6.C, L1.P$1, U$2.SW2
- removed net N$29: C26.2, R18.1
- removed net N$30: C21.2, C27.2, R18.2, R22.2, R25.1, U$2.FB
- removed net N$31: C27.1, R23.1
- removed net N$32: R19.1, U$3.RUN
- removed net N$33: R20.1, U$3.PWM
- removed net N$34: D8.C, L2.P$2, U$3.SW1
- removed net N$35: D5.C, L2.P$1, U$3.SW2
- removed net N$36: C22.1, C23.1, U$3.VC
- removed net N$37: C23.2, R21.1
- removed net N$38: C22.2, C29.2, R21.2, R24.2, R27.1, U$3.FB
- removed net N$39: C29.1, R26.1
- removed net N$40: LED1.C, R28.2
- new net N$22: U$1.40
- net +3V3: now also U$2.VCC1
- net GND: no longer C24.2, C25.2, C28.2, C30.2, POWER_IN1.2, R22.1, R24.1, R28.1, U$2.GND1, U$2.GND2, U$2.GND3, U$2.GND4, U$2.GND5, U$2.PGND1, U$2.PGND2, U$3.GND1, U$3.GND2, U$3.GND3, U$3.GND4, U$3.GND5, U$3.PGND1, U$3.PGND2
- net N$24: now also R17.1, U$2.G4; no longer C21.1, C26.1, U$2.VC
- net N$25: now also U$2.R3; no longer U$2.RUN
- net N$26: now also R18.1, U$2.B2; no longer D7.C, L1.P$2, U$2.SW1
- net N$43: now also R17.2
- net N$46: now also R16.2
- net N$47: now also R18.2
- net V+: no longer C24.1, C25.1, C28.1, C30.1, D5.A, D6.A, D7.A, D8.A, LED1.A, POWER_IN1.1, R16.2, R17.2, R19.2, R20.2, R23.2, R25.2, R26.2, R27.2, U$2.PVI, U$2.VI, U$2.VO, U$3.PVI, U$3.VI, U$3.VO
Other:
- note removed: "4.7uH"
- note removed: "IC3"
- note removed: "IC4"
- note removed: "L1"
- note removed: "L2"
- note removed: "LTC3534"
- note removed: "POWER_BLOCK_A"
- moved on the sheet: C1, C10, C11, C12, C13, C14, C15, C16, C17, C18, C19, C2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
