File: Schematics/LDO/LDO.brd (EAGLE design)
At the start: 100 x 80 mm, 59 parts, among them IC1 LM317MBSTT3, IC2 LM317MBSTT3, Q1 32.768kHz, X1 MINI-USB-SHIELD-UX60-MB-5ST, X2 RJ45

Commit message: LDO Layout
Parts:
- moved C6 142.5 mm to (69.1, 48.0), turned to 270 degrees
- moved C5 141.4 mm to (71.4, 40.1), turned to 270 degrees
- moved Z3 140.6 mm to (79.5, 20.8), turned to 90 degrees
- moved C20 137.7 mm to (81.8, 41.9), turned to 90 degrees
- moved Z2 136.1 mm to (82.3, 20.8), turned to 90 degrees
- moved U$5 133.9 mm to (65.0, 3.05), turned to 180 degrees
- moved Z1 131.4 mm to (84.8, 21.1), turned to 90 degrees
- moved C1 129.9 mm to (62.7, 20.8), turned to 270 degrees
- moved Q1 129.1 mm to (79.8, 45.0)
- moved C2 129.0 mm to (52.1, 39.9)
- moved C19 128.0 mm to (78.2, 41.9), turned to 90 degrees
- moved R6 125.3 mm to (79.5, 30.2), turned to 180 degrees
- moved R10 124.7 mm to (89.7, 22.4), turned to 180 degrees
- moved X1 124.4 mm to (87.4, 33.3), turned to 180 degrees
- moved C13 123.0 mm to (89.9, 18.3), turned to 180 degrees
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Connections:
- removed net AGND: C14.1, C15.1, C3.1, C6.1, U$1.P$23, X2.3
- net GND: now also C14.1, C15.1, C3.1, C6.1, U$1.P$23, X2.3
Routing:
- net +3V3: track 45.4 -> 275.1 mm, vias 0 -> 12
- net GND: track 64.8 -> 189.8 mm, vias 22 -> 69
- net +5V: track 48.3 -> 151.7 mm, vias 0 -> 3
- net N$41: track 0.00 -> 40.3 mm, vias 0 -> 2
- net N$44: track 0.00 -> 38.7 mm, vias 0 -> 4
- net PE: track 0.00 -> 37.3 mm, vias 0 -> 2
- net N$21: track 0.00 -> 32.8 mm, vias 0 -> 3
- net N$19: track 0.00 -> 31.1 mm, vias 0 -> 2
- net N$18: track 0.00 -> 30.9 mm, vias 0 -> 2
- net N$8: track 0.00 -> 30.0 mm, vias 0 -> 3
- net ANALOGINPUT: track 0.00 -> 29.4 mm, vias 0 -> 3
- net N$7: track 0.00 -> 27.6 mm, vias 0 -> 2
- net N$42: track 0.00 -> 27.0 mm, vias 0 -> 2
- net N$20: track 0.00 -> 24.9 mm, vias 0 -> 2
- net N$3: track 0.00 -> 24.6 mm, vias 0 -> 2
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Other:
- board size 100 x 80 mm -> 92.4 x 80.3 mm
- board text added: "OFF"
- board text added: "ON"

Commit message: Layout for final inspection
Parts:
- R9: value 380 -> 383
- moved C5 0.22 mm to (71.3, 39.9)
- renumbered U$2 to D6
Routing:
- net N$7: track 27.6 -> 31.7 mm
Other:
- outline, holes or cut-outs redrawn
- board text added: "B1"
- board text added: "B2"
- board text added: "D10"
- board text added: "Erebus Labs"
- board text added: "Main Board"
- board text added: "Rev 0"

Commit message: PCB Verify Push. Status: In Progress
Routing:
- net GND: vias 69 -> 65
Other:
- board size 92.4 x 80.3 mm -> 92.4 x 80 mm
- board text added: "Ethernet"
- board text added: "Microcontroller"
- board text added: "Programmer"
- board text added: "Regulator 3.3"
- board text added: "Regulator 5V"
- board text added: "START"
- board text added: "STOP"
- board text added: "USB"
- board text removed: "OFF"
- board text removed: "ON"
Changed lines of the file:
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@@
 <?xml version="1.0" encoding="utf-8"?>
 <!DOCTYPE eagle SYSTEM "eagle.dtd">
-<eagle version="6.4">
+<eagle version="6.5.0">
 <drawing>
 <settings>
@@
 <plain>
 <wire x1="0" y1="0" x2="92.38" y2="0.054" width="0" layer="20"/>
-<wire x1="92.38" y1="0.054" x2="92.38" y2="80.254" width="0" layer="20"/>
-<wire x1="92.38" y1="80.254" x2="0" y2="80" width="0" layer="20"/>
+<wire x1="92.38" y1="0.054" x2="92.38" y2="79.954" width="0" layer="20"/>
+<wire x1="92.38" y1="79.954" x2="0" y2="80" width="0" layer="20"/>
 <wire x1="0" y1="80" x2="0" y2="0" width="0" layer="20"/>
 <text x="71.1" y="68.9" size="1.778" layer="25">Erebus Labs</text>
-<text x="71.5" y="66.3" size="1.778" layer="25">Main Board</text>
-<text x="74.7" y="63.7" size="1.778" layer="25">Rev 0</text>
-<text x="47.3" y="4.8" size="1.778" layer="25" rot="R90">ON</text>
-<text x="69.3" y="4.9" size="1.778" layer="25" rot="R90">OFF</text>
+<text x="70.9" y="66.3" size="1.778" layer="25">Main Board</text>
+<text x="71.1" y="63.7" size="1.778" layer="25">Rev 0</text>
+<text x="48.4" y="3.9" size="1.778" layer="25" rot="R180">START</text>
+<text x="73.4" y="3.9" size="1.778" layer="25" rot="R180">STOP</text>
 <text x="53.1" y="29.3" size="0.8128" layer="25" rot="R90">D10</text>
-<text x="50.7" y="2.4" size="1.778" layer="25">B1</text>
-<text x="61.3" y="2.3" size="1.778" layer="25">B2</text>
+<text x="50.5" y="11.6" size="1.778" layer="25">B1</text>
+<text x="61.2" y="11.3" size="1.778" layer="25">B2</text>
+<text x="86.3" y="40.6" size="1.778" layer="25">USB</text>
+<text x="43.5" y="65.2" size="1.778" layer="25">Ethernet</text>
+<text x="53.7" y="29.5" size="1.778" layer="25">Microcontroller</text>
+<text x="10.2" y="32.7" size="1.778" layer="25">Regulator 3.3</text>
+<text x="10.4" y="73.5" size="1.778" layer="25">Regulator 5V</text>
+<text x="63.7" y="13.5" size="1.778" layer="25">Programmer</text>
 </plain>
 <attributes>
@@
 <wire x1="44.958" y1="26.416" x2="44.577" y2="26.797" width="2.54" layer="16"/>
 <via x="44.577" y="26.797" extent="1-16" drill="0.5" diameter="1.27" shape="octagon"/>
-<via x="54.356" y="30.48" extent="1-16" drill="0.5" diameter="0.254" shape="octagon"/>
-<via x="56.642" y="30.734" extent="1-16" drill="0.5" diameter="0.254" shape="octagon"/>
 <via x="62.484" y="29.21" extent="1-16" drill="0.5" diameter="0.254" shape="octagon"/>
 <via x="62.992" y="32.004" extent="1-16" drill="0.5" diameter="0.254" shape="octagon"/>
@@
 <via x="63.5" y="16.764" extent="1-16" drill="0.5" diameter="0.254" shape="octagon"/>
 <via x="68.326" y="11.176" extent="1-16" drill="0.5" diameter="0.254" shape="octagon"/>
-<via x="72.644" y="14.986" extent="1-16" drill="0.5" diameter="0.254" shape="octagon"/>
 <wire x1="89.041" y1="18.288" x2="80.4862" y2="18.288" width="0.4064" layer="1"/>
 <wire x1="80.4862" y1="18.288" x2="79.502" y2="20.0342" width="0.4064" layer="1"/>
@@
 <via x="58.928" y="24.384" extent="1-16" drill="0.5" diameter="0.254"/>
 <via x="62.738" y="24.892" extent="1-16" drill="0.5" diameter="0.254"/>
-<via x="68.326" y="30.988" extent="1-16" drill="0.5" diameter="0.254"/>
 <via x="76.708" y="17.526" extent="1-16" drill="0.5" diameter="0.254"/>
 <via x="75.946" y="20.828" extent="1-16" drill="0.5" diameter="0.254"/>

Commit message: Added Battery Sense to LDO
Parts:
- added R19, R2: 5.6k, rcl:R0805
- H1, H2, H3, H4: value MOUNT-HOLE3.0 -> MOUNT-HOLE2.8; device holes:3,0 -> holes:2,8
Connections:
- new net N$12: R19.2, R2.1, U$1.P$44
- net GND: now also R19.1
- net V+: now also R2.2
Routing:
- net V+: track 102.8 -> 146.5 mm, vias 2 -> 3
- net N$12: track 0.00 -> 23.9 mm
