File: Schematics/Switching/Main_Board_SW.brd (EAGLE design)
At the start: 100 x 80 mm, 83 parts, among them Q1 32.768kHz, X1 MINI-USB-SHIELD-UX60-MB-5ST, X2 RJ45

Commit message: Layout for final inspection
Parts:
- moved U$5 27.3 mm to (61.4, 10.8), turned to 0 degrees
- moved U$6 13.3 mm to (50.4, 11.0), turned to 0 degrees
- moved C20 5.44 mm to (82.8, 38.1)
- moved Q1 4.19 mm to (84.5, 44.1)
- moved C19 4.09 mm to (80.4, 39.5)
- moved H3 2.55 mm to (95.6, 75.8)
- moved H1 2.21 mm to (95.7, 4.50)
- moved H4 1.46 mm to (4.55, 75.7)
- moved H2 1.38 mm to (4.25, 4.50)
Routing:
- net GND: track 498.2 -> 440.6 mm, vias 123 -> 114
- net N$41: track 20.5 -> 50.9 mm, vias 2 -> 4
- net +3V3: track 232.1 -> 260.5 mm, vias 12 -> 14
- net N$44: track 27.4 -> 39.9 mm
- net N$23: track 32.2 -> 25.7 mm
- net N$16: track 36.2 -> 31.4 mm
Other:
- board text added: "B1"
- board text added: "B2"
- board text added: "D10"
- board text added: "Erebus Labs"
- board text added: "Main Board"
- board text added: "OFF"
- board text added: "ON"
- board text added: "Rev 0"
