File: Schematics/Ligth_Sensor/Light_Sensor_Layout.brd (EAGLE design)
At the start: 39 x 40.6 mm, 9 parts, among them J1 RJ45

Commit message: Cleaned up stuff
Made Schematics easier to read
Split Supplies in BOM and made names match references
Renamed parts on sensor
Parts:
- renumbered C1 to C33, C2 to C34, J1 to J2, R1 to R31
Changed lines of the file:
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@@
 <grid distance="0.1" unitdist="mm" unit="mm" style="lines" multiple="1" display="no" altdistance="0.025" altunitdist="inch" altunit="inch"/>
 <layers>
-<layer number="1" name="Top" color="4" fill="1" visible="no" active="yes"/>
-<layer number="16" name="Bottom" color="1" fill="1" visible="no" active="yes"/>
-<layer number="17" name="Pads" color="2" fill="1" visible="no" active="yes"/>
-<layer number="18" name="Vias" color="2" fill="1" visible="no" active="yes"/>
-<layer number="19" name="Unrouted" color="6" fill="1" visible="no" active="yes"/>
+<layer number="1" name="Top" color="4" fill="1" visible="yes" active="yes"/>
+<layer number="16" name="Bottom" color="1" fill="1" visible="yes" active="yes"/>
+<layer number="17" name="Pads" color="2" fill="1" visible="yes" active="yes"/>
+<layer number="18" name="Vias" color="2" fill="1" visible="yes" active="yes"/>
+<layer number="19" name="Unrouted" color="6" fill="1" visible="yes" active="yes"/>
 <layer number="20" name="Dimension" color="15" fill="1" visible="yes" active="yes"/>
 <layer number="21" name="tPlace" color="7" fill="1" visible="yes" active="yes"/>
-<layer number="22" name="bPlace" color="7" fill="1" visible="no" active="yes"/>
-<layer number="23" name="tOrigins" color="15" fill="1" visible="no" active="yes"/>
-<layer number="24" name="bOrigins" color="15" fill="1" visible="no" active="yes"/>
-<layer number="25" name="tNames" color="7" fill="1" visible="no" active="yes"/>
-<layer number="26" name="bNames" color="7" fill="1" visible="no" active="yes"/>
-<layer number="27" name="tValues" color="7" fill="1" visible="no" active="yes"/>
-<layer number="28" name="bValues" color="7" fill="1" visible="no" active="yes"/>
+<layer number="22" name="bPlace" color="7" fill="1" visible="yes" active="yes"/>
+<layer number="23" name="tOrigins" color="15" fill="1" visible="yes" active="yes"/>
+<layer number="24" name="bOrigins" color="15" fill="1" visible="yes" active="yes"/>
+<layer number="25" name="tNames" color="7" fill="1" visible="yes" active="yes"/>
+<layer number="26" name="bNames" color="7" fill="1" visible="yes" active="yes"/>
+<layer number="27" name="tValues" color="7" fill="1" visible="yes" active="yes"/>
+<layer number="28" name="bValues" color="7" fill="1" visible="yes" active="yes"/>
 <layer number="29" name="tStop" color="7" fill="3" visible="no" active="yes"/>
 <layer number="30" name="bStop" color="7" fill="6" visible="no" active="yes"/>
@@
 <layer number="42" name="bRestrict" color="1" fill="10" visible="no" active="yes"/>
 <layer number="43" name="vRestrict" color="2" fill="10" visible="no" active="yes"/>
-<layer number="44" name="Drills" color="7" fill="1" visible="yes" active="yes"/>
-<layer number="45" name="Holes" color="7" fill="1" visible="yes" active="yes"/>
+<layer number="44" name="Drills" color="7" fill="1" visible="no" active="yes"/>
+<layer number="45" name="Holes" color="7" fill="1" visible="no" active="yes"/>
 <layer number="46" name="Milling" color="3" fill="1" visible="no" active="yes"/>
 <layer number="47" name="Measures" color="7" fill="1" visible="yes" active="yes"/>
-<layer number="48" name="Document" color="7" fill="1" visible="no" active="yes"/>
-<layer number="49" name="Reference" color="7" fill="1" visible="no" active="yes"/>
-<layer number="51" name="tDocu" color="7" fill="1" visible="no" active="yes"/>
-<layer number="52" name="bDocu" color="7" fill="1" visible="no" active="yes"/>
+<layer number="48" name="Document" color="7" fill="1" visible="yes" active="yes"/>
+<layer number="49" name="Reference" color="7" fill="1" visible="yes" active="yes"/>
+<layer number="51" name="tDocu" color="7" fill="1" visible="yes" active="yes"/>
+<layer number="52" name="bDocu" color="7" fill="1" visible="yes" active="yes"/>
 <layer number="91" name="Nets" color="2" fill="1" visible="no" active="no"/>
 <layer number="92" name="Busses" color="1" fill="1" visible="no" active="no"/>
@@
 <text x="11.43" y="73.66" size="1.778" layer="21">Light Sensor </text>
 <text x="11.43" y="71.12" size="1.778" layer="21">Rev 0</text>
-<dimension x1="0" y1="80" x2="5.08" y2="74.93" x3="2.54" y3="74.93" textsize="1.778" layer="20" dtype="horizontal"/>
-<dimension x1="33" y1="75" x2="39" y2="75" x3="36" y3="75" textsize="1.778" layer="20" dtype="horizontal"/>
-<dimension x1="33.1" y1="44.4" x2="39" y2="43.7" x3="36.05" y3="44.5" textsize="1.778" layer="20" dtype="horizontal"/>
-<dimension x1="5" y1="44.5" x2="0" y2="43.6" x3="2.5" y3="44.5" textsize="1.778" layer="20" dtype="horizontal"/>
-<dimension x1="0" y1="39.37" x2="39" y2="41.3" x3="19.5" y3="35.7" textsize="1.778" layer="20" dtype="horizontal"/>
-<dimension x1="5" y1="74.9" x2="3.6" y2="80" x3="5" y3="77.45" textsize="1.778" layer="20" dtype="vertical"/>
-<dimension x1="33.1" y1="74.9" x2="31.8" y2="80" x3="33" y3="77.45" textsize="1.778" layer="20" dtype="vertical"/>
-<dimension x1="33" y1="44.5" x2="31.5" y2="39.4" x3="33" y3="41.95" textsize="1.778" layer="20" dtype="vertical"/>
-<dimension x1="5" y1="44.5" x2="7.9" y2="39.3" x3="5" y3="41.9" textsize="1.778" layer="20" dtype="vertical"/>
-<dimension x1="39.04" y1="80" x2="39.04" y2="39.37" x3="44.8" y3="59.685" textsize="1.778" layer="20" dtype="vertical"/>
-<dimension x1="13.8" y1="65.9" x2="14.4" y2="80" x3="28.7" y3="72.95" textsize="1.778" layer="20" dtype="vertical"/>
-<dimension x1="13.6" y1="50.9" x2="12.8" y2="39.4" x3="13.3" y3="45.15" textsize="1.778" layer="20" dtype="vertical"/>
 </plain>
 <attributes>
@@
 <attribute name="NAME" x="29.21" y="55.88" size="1.27" layer="25"/>
 </element>
-<element name="R1" library="rcl" package="R1206" value="10k" x="26.035" y="48.895" smashed="yes" rot="R90">
+<element name="R31" library="rcl" package="R1206" value="10k" x="26.035" y="48.895" smashed="yes" rot="R90">
 <attribute name="NAME" x="29.845" y="50.165" size="1.27" layer="25" rot="R180"/>
 <attribute name="VALUE" x="29.845" y="48.26" size="1.27" layer="27" rot="R180"/>
 </element>
-<element name="J1" library="con-amp" package="555167-1" value="RJ45" x="6.35" y="58.42" rot="R270"/>
+<element name="J2" library="con-amp" package="555167-1" value="RJ45" x="6.35" y="58.42" rot="R270"/>
 <element name="H1" library="holes" package="2,8" value="MOUNT-HOLE2.8" x="5.08" y="44.45"/>
 <element name="H2" library="holes" package="2,8" value="MOUNT-HOLE2.8" x="33.02" y="44.45"/>
 <element name="H3" library="holes" package="2,8" value="MOUNT-HOLE2.8" x="33.02" y="74.93"/>
 <element name="H4" library="holes" package="2,8" value="MOUNT-HOLE2.8" x="5.08" y="74.93"/>
-<element name="C1" library="rcl" package="C0603K" value="0.1uF" x="19.685" y="58.42" rot="R180"/>
-<element name="C2" library="rcl" package="C0603K" value="0.1uF" x="19.685" y="55.88" rot="R180"/>
+<element name="C33" library="rcl" package="C0603K" value="0.1uF" x="19.685" y="58.42" smashed="yes" rot="R180">
+<attribute name="NAME" x="20.485" y="57.77" size="1.016" layer="25" rot="R180"/>
+<attribute name="VALUE" x="21.23" y="60.285" size="1.016" layer="27" rot="R270"/>
+</element>
+<element name="C34" library="rcl" package="C0603K" value="0.1uF" x="19.685" y="55.88" smashed="yes" rot="R180">
+<attribute name="NAME" x="20.485" y="55.23" size="1.016" layer="25" rot="R180"/>
+<attribute name="VALUE" x="21.17" y="56.385" size="1.016" layer="27" rot="R270"/>
+</element>
 </elements>
 <signals>
 <signal name="N$1">
 <contactref element="PH1" pad="1"/>
-<contactref element="J1" pad="4"/>
+<contactref element="J2" pad="4"/>
 <wire x1="14.097" y1="59.055" x2="15.875" y2="59.055" width="0.8128" layer="1"/>
 <wire x1="15.875" y1="59.055" x2="17.78" y2="60.96" width="0.8128" layer="1"/>
@@
 <signal name="N$2">
 <contactref element="PH1" pad="2"/>
-<contactref element="R1" pad="2"/>
-<contactref element="J1" pad="7"/>
+<contactref element="R31" pad="2"/>
+<contactref element="J2" pad="7"/>
 <wire x1="11.557" y1="55.245" x2="16.51" y2="55.245" width="0.8128" layer="1"/>
 <wire x1="26.035" y1="55.245" x2="26.035" y2="52.705" width="0.8128" layer="1"/>
@@
 </signal>
 <signal name="AGND">
-<contactref element="R1" pad="1"/>
+<contactref element="R31" pad="1"/>
 <polygon width="0.4064" layer="16">
 <vertex x="0" y="80.01"/>
@@
 <vertex x="0" y="39.37"/>
 </polygon>
-<contactref element="J1" pad="8"/>
-<contactref element="J1" pad="1"/>
-<contactref element="J1" pad="2"/>
-<contactref element="J1" pad="3"/>
-<contactref element="C1" pad="1"/>
-<contactref element="C2" pad="1"/>
+<contactref element="J2" pad="8"/>
 <via x="20.32" y="41.91" extent="1-16" drill="0.6" diameter="0.4064"/>
 <via x="15.24" y="45.72" extent="1-16" drill="0.6" diameter="0.4064"/>
@@
 <via x="27.94" y="77.47" extent="1-16" drill="0.6" diameter="0.4064"/>
 <via x="26.67" y="73.025" extent="1-16" drill="0.6" diameter="0.4064"/>
+<contactref element="J2" pad="1"/>
+<contactref element="J2" pad="2"/>
+<contactref element="J2" pad="3"/>
+<contactref element="C33" pad="1"/>
+<contactref element="C34" pad="1"/>
 </signal>
 <signal name="N$16">
 </signal>
 <signal name="N$23">
-<contactref element="J1" pad="5"/>
-<contactref element="C1" pad="2"/>
+<contactref element="J2" pad="5"/>
+<contactref element="C33" pad="2"/>
 <wire x1="11.557" y1="57.785" x2="16.51" y2="57.785" width="0.8128" layer="1"/>
 <wire x1="16.51" y1="57.785" x2="17.145" y2="58.42" width="0.8128" layer="1"/>
@@
 </signal>
 <signal name="N$24">
-<contactref element="J1" pad="6"/>
-<contactref element="C2" pad="2"/>
+<contactref element="J2" pad="6"/>
+<contactref element="C34" pad="2"/>
 <wire x1="14.097" y1="56.515" x2="17.145" y2="56.515" width="0.8128" layer="1"/>
 <wire x1="17.145" y1="56.515" x2="17.78" y2="55.88" width="0.8128" layer="1"/>
